File: PAWPAD/PAWPAD.kicad_pcb (KiCad board)
At the start: 2 copper layers, 42.3 x 42 mm, 29 parts, among them J1 Conn_01x01, J2 Conn_01x01, J3 Conn_01x01, J4 Conn_01x01, J5 Conn_01x01, U1 AT42QT1070-S

Commit message: update silkscreen
Parts:
- added REF**: OSHW-Logo_5.7x6mm_SilkScreen, Symbol:OSHW-Logo_5.7x6mm_SilkScreen, B.Cu at (167.0, 102.9)
- added Ref**: Val**, random stuff:mothface, B.Cu at (152.4, 85.3)
Other:
- board text added: "made by eri CC-BY-SA moth.monster"
- board text removed: "CC-BY-SA"
- board text removed: "made by eri"
