File: atx breakout/atx breakout.kicad_pcb (KiCad board)
At the start: 2 copper layers, 53.3 x 44.5 mm, 15 parts, among them J1 ATX-20, J2 ON/OFF, J3 12V, J4 5V, J5 3.3V, SW1 SW_Push

Commit message: fix switch
Parts:
- SW1: value SW_Push -> SW_SPST; footprint Button_Switch_THT:SW_PUSH_6mm -> Connector_PinHeader_2.54mm:PinHeader_1x03_P2.54mm_Vertical
- moved SW1 2.36 mm to (133.3, 85.1), turned to -90 degrees
Connections:
- net /12V renamed Net-(D2-Pad2)
- net /3.3V renamed Net-(D4-Pad2)
- net /5V renamed Net-(D3-Pad2)
- net /GND renamed Net-(J1-Pad13)
Routing:
- net Net-(J1-Pad13): track 0.00 -> 13.9 mm
- net Net-(J1-Pad14): track 39.2 -> 39.9 mm
