File: atx breakout/atx breakout.kicad_sch (KiCad schematic)
At the start: 14 parts, among them J1 ATX-20, J2 ON/OFF, J3 12V, J4 5V, J5 3.3V, SW1 SW_Push

Commit message: fix switch
Parts:
- removed SW1: SW_Push, Button_Switch_THT:SW_PUSH_6mm, symbol Switch:SW_Push
- added SW1: SW_SPST, Connector_PinHeader_2.54mm:PinHeader_1x03_P2.54mm_Vertical, symbol Switch:SW_SPST
Connections:
- net at J1.13 (GND), J1.15 (GND), J1.16 (GND)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: now also SW1.1 (A)
- net at J1.14 (PS_ON#), J2.1 (Pin_1): now also SW1.2 (B)
Changed lines of the file:
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@@
 (kicad_sch (version 20210406) (generator eeschema)
   (paper "A4")
-  (junction (at 120.65 73.66) (diameter 1.016) (color 0 0 0 0))
-  (junction (at 120.65 83.82) (diameter 1.016) (color 0 0 0 0))
+  (junction (at 91.44 73.66) (diameter 1.016) (color 0 0 0 0))
   (junction (at 120.65 85.09) (diameter 1.016) (color 0 0 0 0))
   (junction (at 120.65 91.44) (diameter 1.016) (color 0 0 0 0))
@@
   (junction (at 154.94 88.9) (diameter 1.016) (color 0 0 0 0))
   (junction (at 154.94 95.25) (diameter 1.016) (color 0 0 0 0))
+  (wire (pts (xy 91.44 68.58) (xy 91.44 73.66))
+    (stroke (width 0) (type solid) (color 0 0 0 0))
+  )
   (wire (pts (xy 91.44 73.66) (xy 91.44 77.47))
     (stroke (width 0) (type solid) (color 0 0 0 0))
   )
+  (wire (pts (xy 91.44 73.66) (xy 121.92 73.66))
+    (stroke (width 0) (type solid) (color 0 0 0 0))
+  )
   (wire (pts (xy 104.14 102.87) (xy 120.65 102.87))
     (stroke (width 0) (type solid) (color 0 0 0 0))
@@
     (stroke (width 0) (type solid) (color 0 0 0 0))
   )
-  (wire (pts (xy 120.65 73.66) (xy 91.44 73.66))
+  (wire (pts (xy 120.65 68.58) (xy 91.44 68.58))
+    (stroke (width 0) (type solid) (color 0 0 0 0))
+  )
+  (wire (pts (xy 120.65 78.74) (xy 120.65 85.09))
     (stroke (width 0) (type solid) (color 0 0 0 0))
   )
@@
     (stroke (width 0) (type solid) (color 0 0 0 0))
   )
-  (wire (pts (xy 120.65 83.82) (xy 120.65 78.74))
-    (stroke (width 0) (type solid) (color 0 0 0 0))
-  )
-  (wire (pts (xy 120.65 85.09) (xy 120.65 83.82))
-    (stroke (width 0) (type solid) (color 0 0 0 0))
-  )
   (wire (pts (xy 120.65 85.09) (xy 120.65 91.44))
     (stroke (width 0) (type solid) (color 0 0 0 0))
@@
   )
   (wire (pts (xy 120.65 102.87) (xy 120.65 97.79))
-    (stroke (width 0) (type solid) (color 0 0 0 0))
-  )
-  (wire (pts (xy 121.92 73.66) (xy 120.65 73.66))
     (stroke (width 0) (type solid) (color 0 0 0 0))
   )
@@
     (pin "2")
   )
+  (symbol (lib_id "Switch:SW_SPST") (at 120.65 73.66 90) (unit 1)
+    (in_bom yes) (on_board yes) (fields_autoplaced)
+    (property "Reference" "SW1" (id 0) (at 121.7931 72.8991 90)
+      (effects (font (size 1.27 1.27)) (justify right))
+    )
+    (property "Value" "SW_SPST" (id 1) (at 121.7931 75.1978 90)
+      (effects (font (size 1.27 1.27)) (justify right))
+    )
+    (property "Footprint" "Connector_PinHeader_2.54mm:PinHeader_1x03_P2.54mm_Vertical" (id 2) (at 120.65 73.66 0)
+      (effects (font (size 1.27 1.27)) hide)
+    )
+    (property "Datasheet" "~" (id 3) (at 120.65 73.66 0)
+      (effects (font (size 1.27 1.27)) hide)
+    )
+    (pin "1")
+    (pin "2")
+  )
   (symbol (lib_id "Device:LED") (at 143.51 76.2 180) (unit 1)
     (in_bom yes) (on_board yes)
@@
     )
     (property "Datasheet" "~" (id 3) (at 127 95.25 0)
-      (effects (font (size 1.27 1.27)) hide)
-    )
-    (pin "1")
-    (pin "2")
-  )
-  (symbol (lib_id "Switch:SW_Push") (at 120.65 78.74 90) (unit 1)
-    (in_bom yes) (on_board yes)
-    (property "Reference" "SW1" (id 0) (at 121.8692 78.74 90)
-      (effects (font (size 1.27 1.27)) (justify right) hide)
-    )
-    (property "Value" "SW_Push" (id 1) (at 121.8692 79.883 90)
-      (effects (font (size 1.27 1.27)) (justify right) hide)
-    )
-    (property "Footprint" "Button_Switch_THT:SW_PUSH_6mm" (id 2) (at 115.57 78.74 0)
-      (effects (font (size 1.27 1.27)) hide)
-    )
-    (property "Datasheet" "~" (id 3) (at 115.57 78.74 0)
       (effects (font (size 1.27 1.27)) hide)
     )
@@
       (reference "R4") (unit 1) (value "47") (footprint "Resistor_THT:R_Axial_DIN0207_L6.3mm_D2.5mm_P10.16mm_Horizontal")
     )
-    (path "/00000000-0000-0000-0000-00006081f8ca"
-      (reference "SW1") (unit 1) (value "SW_Push") (footprint "Button_Switch_THT:SW_PUSH_6mm")
-    )
-  )
+    (path "/848abd4e-45c6-451e-b927-2e54feda722f"
+      (reference "SW1") (unit 1) (value "SW_SPST") (footprint "Connector_PinHeader_2.54mm:PinHeader_1x03_P2.54mm_Vertical")
+    )
+  )
